Commit message: update sample of mid360

File: robots/descriptions/go2_description/xacro/mid360.xacro (robot description, xacro)
@@ -4,5 +4,5 @@
   <xacro:property name="laser_min_range" value="0.1"/>
   <xacro:property name="laser_max_range" value="100.0"/>
-  <xacro:property name="samples" value="40000"/>
+  <xacro:property name="samples" value="20000"/>
   <xacro:property name="resolution" value="0.002"/>
   <xacro:property name="noise_mean" value="0.0"/>
